Commit message: simplified code to make it easier to test

File: catkin_ws/src/autonomous_drone/plugins/bodyNsensors.urdf.xacro (robot description, xacro)
@@ -41,14 +41,2 @@
   </xacro:macro>
     <quadrotor_base_body />
-<!-- //////////////////////// Seperated from main body and generic quadrotor plugins  //////////////////////////-->
-    <!-- Hokuyo Laser sensor gazebo plugin  -->
-    <xacro:include filename="$(find autonomous_drone)/sensors/hokuyo_utm30lx.urdf.xacro" />
-    <xacro:hokuyo_utm30lx name="laser" parent="base_link" ros_topic="scan" update_rate="40" ray_count="1081" min_angle="135" max_angle="-135">
-      <origin xyz="0.0 0.0 0.08" rpy="3.14 0 0"/>
-    </xacro:hokuyo_utm30lx>
-    <!-- Hokuyo Laser sensor gazebo plugin  -->
-        <xacro:include filename="$(find autonomous_drone)/sensors/sonar_sensor.urdf.xacro" />
-    <xacro:sonar_sensor name="sonar" parent="base_link" ros_topic="sonar_height" update_rate="10" min_range="0.01" max_range="3.0" field_of_view="${40*M_PI/180}" ray_count="3">
-      <origin xyz="-0.15 0.0 0.0" rpy="0 ${90*M_PI/180} 0"/>
-    </xacro:sonar_sensor>
-</robot>

Commit message: Added code to implement sensors that will be reading the environment

File: catkin_ws/src/autonomous_drone/plugins/bodyNsensors.urdf.xacro (robot description, xacro)
@@ -41,3 +41,14 @@
   </xacro:macro>
     <quadrotor_base_body/>
+    <!-- //////////////////////// Seperated from main body and generic quadrotor plugins  //////////////////////////-->
+    <!-- Hokuyo Laser sensor gazebo plugin  -->
+    <xacro:include filename="$(find autonomous_drone)/sensors/hokuyo_utm30lx.urdf.xacro" />
+    <xacro:hokuyo_utm30lx name="laser" parent="base_link" ros_topic="scan" update_rate="40" ray_count="1081" min_angle="135" max_angle="-135">
+      <origin xyz="0.0 0.0 0.08" rpy="3.14 0 0"/>
+    </xacro:hokuyo_utm30lx>
+    <!-- Hokuyo Laser sensor gazebo plugin  -->
+        <xacro:include filename="$(find autonomous_drone)/sensors/sonar_sensor.urdf.xacro" />
+    <xacro:sonar_sensor name="sonar" parent="base_link" ros_topic="sonar_height" update_rate="10" min_range="0.01" max_range="3.0" field_of_view="${40*M_PI/180}" ray_count="3">
+      <origin xyz="-0.15 0.0 0.0" rpy="0 ${90*M_PI/180} 0"/>
+    </xacro:sonar_sensor>
 </robot>
