Commit message: Editied launch file to include new world for drone to navigate

File: catkin_ws/src/autonomous_drone/plugins/DroneAndSensors.urdf.xacro (robot description, xacro)
@@ -1,4 +1,4 @@
 <?xml version="1.0"?>
-<robot name="myquadrotor"
+<robot name="mydrone"
 xmlns:sensor="http://playerstage.sourceforge.net/gazebo/xmlschema/#sensor"
 xmlns:controller="http://playerstage.sourceforge.net/gazebo/xmlschema/#controller"
@@ -15,10 +15,10 @@
   <xacro:include filename="$(find autonomous_drone)/plugins/gazebo_sim_controller.urdf.xacro" />
   <!-- Main body link -->
-  <xacro:macro name="quadrotor_base_body">
+  <xacro:macro name="drone_base_body">
     <link name="base_link">
       <inertial>
-        <mass value="1.477" />
+        <mass value="1.233" />
         <origin xyz="0 0 0" />
-        <inertia ixx="0.01152" ixy="0.0" ixz="0.0" iyy="0.01152" iyz="0.0" izz="0.0218" />
+        <inertia ixx="0.01153" ixy="0.0" ixz="0.0" iyy="0.01153" iyz="0.0" izz="0.0219" />
       </inertial>
       <visual>

Commit message: added comments to code

File: catkin_ws/src/autonomous_drone/plugins/DroneAndSensors.urdf.xacro (robot description, xacro)
@@ -14,5 +14,5 @@
   <xacro:include filename="$(find autonomous_drone)/plugins/gazebo_sim_plugins.urdf.xacro" />
   <xacro:include filename="$(find autonomous_drone)/plugins/gazebo_sim_controller.urdf.xacro" />
-  <!-- Main body link -->
+  <!-- Main body of the drone information -->
   <xacro:macro name="drone_base_body">
     <link name="base_link">
@@ -42,13 +42,13 @@
     <quadrotor_base_body/>
     <!-- //////////////////////// Seperated from main body and generic quadrotor plugins  //////////////////////////-->
-    <!-- Hokuyo Laser sensor gazebo plugin  -->
+    <!-- sonar sensor gazebo plugin implementation  -->
+        <xacro:include filename="$(find autonomous_drone)/sensors/sonar_sensor.urdf.xacro" />
+    <xacro:sonar_sensor name="sonar" parent="base_link" ros_topic="sonar_height" update_rate="10" min_range="0.01" max_range="3.0" field_of_view="${40*M_PI/180}" ray_count="3">
+      <origin xyz="-0.15 0.0 0.0" rpy="0 ${90*M_PI/180} 0"/>
+    </xacro:sonar_sensor>
+    <!-- Hokuyo Laser sensor gazebo plugin implmenetation -->
     <xacro:include filename="$(find autonomous_drone)/sensors/hokuyo_utm30lx.urdf.xacro" />
     <xacro:hokuyo_utm30lx name="laser" parent="base_link" ros_topic="scan" update_rate="40" ray_count="1081" min_angle="135" max_angle="-135">
       <origin xyz="0.0 0.0 0.08" rpy="3.14 0 0"/>
     </xacro:hokuyo_utm30lx>
-    <!-- Hokuyo Laser sensor gazebo plugin  -->
-        <xacro:include filename="$(find autonomous_drone)/sensors/sonar_sensor.urdf.xacro" />
-    <xacro:sonar_sensor name="sonar" parent="base_link" ros_topic="sonar_height" update_rate="10" min_range="0.01" max_range="3.0" field_of_view="${40*M_PI/180}" ray_count="3">
-      <origin xyz="-0.15 0.0 0.0" rpy="0 ${90*M_PI/180} 0"/>
-    </xacro:sonar_sensor>
 </robot>
